File: picofusion_jig_hw.kicad_pcb (KiCad board)
At the start: 2 copper layers, 65 parts, among them J1 PICO_WEST, J10 TELEM, J11 DEBUG, J12 IMU_DBG, J13 NORTH, J14 EAST, J15 SOUTH, J16 WEST, J17 CAN, J2 PICO_EAST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

Commit message: Layout draft
Parts:
- added C3: 0.1uF, Capacitor_SMD:C_0603_1608Metric, F.Cu at (85.8, 104.8)
- added C4: 0.1uF, Capacitor_SMD:C_0603_1608Metric, F.Cu at (82.3, 101.9)
- added C5: 0.1uF, Capacitor_SMD:C_0603_1608Metric, F.Cu at (100.0, 104.8)
- added C6: 0.1uF, Capacitor_SMD:C_0603_1608Metric, F.Cu at (96.7, 101.9)
- BZ1: footprint Resistor_SMD:R_0603_1608Metric -> Buzzer_Beeper:Buzzer_Murata_PKMCS0909E
- J1, J2: footprint Connector_PinSocket_2.54mm:PinSocket_1x20_P2.54mm_Vertical -> Connector_PinSocket_2.54mm:PinSocket_1x20_P2.54mm_Vertical_SMD_Pin1Left
- moved J7 109.6 mm to (146.3, 109.4), turned to 90 degrees
- moved J13 101.8 mm to (129.0, 75.5)
- moved J14 101.8 mm to (141.0, 87.5)
- moved J15 101.8 mm to (129.0, 99.5)
- moved J16 101.8 mm to (117.0, 87.5)
- moved J10 97.6 mm to (131.6, 121.3)
- moved J1 94.7 mm to (54.0, 87.5)
- moved J2 94.7 mm to (71.8, 87.5)
- moved J9 86.3 mm to (137.4, 51.8), turned to 180 degrees
- moved R20 83.9 mm to (134.2, 71.8), turned to 180 degrees
- moved Q1 81.9 mm to (136.6, 110.4)
- moved J5 79.7 mm to (66.4, 118.0)
- moved SW2 79.6 mm to (108.9, 55.9)
- moved Q2 76.7 mm to (126.6, 110.4)
- moved R11 75.8 mm to (103.6, 111.3), turned to -90 degrees
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Connections:
- C1 pad 2: Net-(C1-Pad2) -> +5V
- J2 pad 17: /UART_RX_GNSS -> /BUZZER
- J2 pad 19: /UART_TX_GNSS -> /UART_RX_GNSS
- J2 pad 20: /BUZZER -> /UART_TX_GNSS
- U3 pad 1: Net-(C1-Pad2) -> +5V
Routing:
- net /UART_TX_TELEM: track 0.00 -> 132.1 mm, vias 0 -> 3
- net /UART_CTS_TELEM: track 0.00 -> 127.6 mm, vias 0 -> 4
- net /UART_RX_TELEM: track 0.00 -> 127.2 mm, vias 0 -> 2
- net /CAN_N: track 0.00 -> 125.9 mm, vias 0 -> 3
- net /CAN_P: track 0.00 -> 122.1 mm, vias 0 -> 3
- net /UART_RX_GNSS: track 0.00 -> 107.1 mm, vias 0 -> 1
- net /UART_TX_GNSS: track 0.00 -> 102.7 mm, vias 0 -> 1
- net /SPI_PICO_SD: track 0.00 -> 98.0 mm, vias 0 -> 2
- net /SPI_POCI_SD: track 0.00 -> 95.4 mm, vias 0 -> 2
- net /IMU_HEATER: track 0.00 -> 91.7 mm, vias 0 -> 2
- net /BUZZER: track 0.00 -> 84.5 mm, vias 0 -> 3
- net /SPI_nCS_SD: track 0.00 -> 78.1 mm, vias 0 -> 1
- net /SDA/SDI: track 0.00 -> 76.6 mm
- net /SD_nCD: track 0.00 -> 73.6 mm, vias 0 -> 1
- net /POCI: track 0.00 -> 67.1 mm
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Other:
- board outline added: 100 x 75 mm
