File: picofusion_jig_hw.kicad_sch (KiCad schematic)
At the start: 65 parts, among them J1 PICO_WEST, J10 TELEM, J11 DEBUG, J12 IMU_DBG, J13 NORTH, J14 EAST, J15 SOUTH, J16 WEST, J17 CAN, J2 PICO_EAST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

Commit message: Layout draft
Parts:
- added C3, C4, C5, C6: 0.1uF, Capacitor_SMD:C_0603_1608Metric, symbol Device:C
- BZ1: footprint Resistor_SMD:R_0603_1608Metric -> Buzzer_Beeper:Buzzer_Murata_PKMCS0909E
- J1, J2: footprint Connector_PinSocket_2.54mm:PinSocket_1x20_P2.54mm_Vertical -> Connector_PinSocket_2.54mm:PinSocket_1x20_P2.54mm_Vertical_SMD_Pin1Left
- J13, J14, J15, J16: footprint Connector_PinHeader_2.54mm:PinHeader_1x08_P2.54mm_Vertical -> picofusion_stamp:Castellated_1x8_P2.54mm_Vertical
Connections:
- net +3V3: now also C3.1, C5.1
- net +5V: now also C1.2, U3.1 (VIN), C4.1, C6.1
- net BUZZER: now also J2.17 (Pin_17); no longer J2.20 (Pin_20)
- net GND: now also C3.2, C4.2, C5.2, C6.2
- net UART_RX_GNSS: now also J2.19 (Pin_19); no longer J2.17 (Pin_17)
- net UART_TX_GNSS: now also J2.20 (Pin_20); no longer J2.19 (Pin_19)
